Commit message: updated the urdf, spawn angle, ros2 integration

File: so101_description/urdf/so101.urdf (robot description, URDF)
Before this commit: robot so101_new_calib, 9 links, 8 joints
Links:
- added link world
- link gripper_frame_link: mass 1e-9 -> 1e-6
Joints:
- added joint base_to_world: type fixed, parent world, child base_link, origin xyz=-0.55 0.0 0.7774 rpy=0 0 0
- joint wrist_roll: origin xyz=5.55112e-17 -0.0611 0.0181 rpy=1.5708 0.0486795 3.14159 -> xyz=5.55112e-17 -0.0611 0.0181 rpy=-1.5708 1.5221132 -7.81e-05
